Commit message: 1

File: test.urdf (robot description, URDF)
Before this commit: robot 天工焊接机器人, 1 links, 0 joints
Links:
- added link Link1; collision mesh filename=meshes/Link1.STL; visual mesh filename=meshes/Link1.STL
Joints:
- added joint joint1: type prismatic, parent base_link, child Link1, origin xyz=-0.5 0.001 0.02 rpy=0 0 1.5708, axis 0 1 0, limit lower=0 upper=14 effort=0 velocity=0

File: tiangong.urdf (robot description, URDF)
Before this commit: robot 天工焊接机器人, 15 links, 14 joints
Links:
- removed link link1-2
- removed link link1-6
- added link Link1-0; collision mesh filename=meshes/Link1-0.STL; visual mesh filename=meshes/Link1-0.STL
- added link Link1-2; collision mesh filename=meshes/Link1-2.STL; visual mesh filename=meshes/Link1-2.STL
- added link Link1-6; collision mesh filename=meshes/Link1-6.STL; visual mesh filename=meshes/Link1-6.STL
- added link Link2-0; collision mesh filename=meshes/Link2-0.STL; visual mesh filename=meshes/Link2-0.STL
- link Link1: mass 2256.89408172069 -> None
- link Link1-1: mass 14468.3356929364 -> None
- link Link1-3: mass 14468.3356929364 -> None
- link Link1-4: mass 14468.3356929364 -> None
- link Link1-5: mass 14468.3356929364 -> None
- link Link2: mass 2523.14851379735 -> None
- link Link2-1: mass 14468.3356929364 -> None
- link Link2-2: mass 14468.3356929364 -> None
- link Link2-3: mass 14468.3356929364 -> None
- link Link2-4: mass 14468.3356929364 -> None
- link Link2-5: mass 14468.3356929364 -> None
- link Link2-6: mass 14468.3356929364 -> None
- link base_link: mass 14468.3356938544 -> None
Joints:
- added joint joint1-0: type prismatic, parent Link1, child Link1-0, origin xyz=-0.0057039 3.1015 -2.5569 rpy=-1.5708 0 -1.5708, axis 1 0 0, limit lower=0 upper=1.7 effort=0 velocity=0
- added joint joint2-0: type prismatic, parent Link2, child Link2-0, origin xyz=0 4.3248 -0.646 rpy=-1.5708 0 -1.5708, axis 1 0 0, limit lower=0 upper=1.7 effort=100 velocity=10
- joint joint1: axis 0 1 0 -> 1 0 0; limit lower=-10 upper=20 effort=0 velocity=0 -> lower=0 upper=14 effort=0 velocity=0; origin xyz=-9.3086 0.0018683 0.02 rpy=0 0 1.5708 -> xyz=-0.0018683 -0.5 0.02 rpy=3.1416 0 -1.5708
- joint joint1-1: limit lower=-3.14 upper=3.14 effort=100 velocity=1 -> lower=-3.14 upper=3.14 effort=100 velocity=10; origin xyz=3.1557 -0.01 2.16 rpy=-1.5708 0 -1.5708 -> xyz=-0.0099737 -0.6255 0.0057037 rpy=0 1.22 3.1416; parent Link1 -> Link1-0
- joint joint1-2: child link1-2 -> Link1-2; limit lower=-3.14 upper=3.14 effort=100 velocity=1 -> lower=-3.14 upper=3.14 effort=100 velocity=10; origin xyz=4.2993 3.9617 1.5934 rpy=-3.1416 0.2601 0.31384 -> xyz=-0.038003 0.242 0.18 rpy=0 0.0074575 -1.5708; parent Link1 -> Link1-1
- joint joint1-3: axis -1 0 0 -> 0 -1 0; limit lower=-3.14 upper=3.14 effort=100 velocity=1 -> lower=-3.14 upper=3.14 effort=100 velocity=10; origin xyz=3.2493 -0.01464 0.91851 rpy=-3.0238 0 -1.257 -> xyz=0 -0.008 0.8 rpy=0 -1.4541 0; parent Link1 -> Link1-2
- joint joint1-4: limit lower=-3.14 upper=3.14 effort=100 velocity=1 -> lower=-3.14 upper=3.14 effort=100 velocity=10; origin xyz=3.6709 0.57585 -0.3882 rpy=0.32676 -0.11777 0.31384 -> xyz=0.0835 0.0433 0.225 rpy=-3.0285 0 0; parent Link1 -> Link1-3
- joint joint1-5: limit lower=-3.14 upper=3.14 effort=100 velocity=1 -> lower=-3.14 upper=3.14 effort=100 velocity=10; origin xyz=2.8979 -0.22313 1.0446 rpy=1.031 1.1901 1.3513 -> xyz=0.9265 -0.0353 0 rpy=0 1.4836 0; parent Link1 -> Link1-4
- joint joint1-6: child link1-6 -> Link1-6; limit lower=-3.14 upper=3.14 effort=100 velocity=1 -> lower=-3.14 upper=3.14 effort=100 velocity=10; origin xyz=4.1216 0.34733 0.7012 rpy=-1.3672 -1.1901 -1.7903 -> xyz=0.0940000046417269 0.0353002689417377 0 rpy=-0.367334218169828 0 -3.14159256129931; parent Link1 -> Link1-5
- joint joint2: axis 0 1 0 -> 1 0 0; limit lower=-20 upper=20 effort=0 velocity=0 -> lower=-25 upper=0 effort=100 velocity=10; origin xyz=-15.745 -0.0099585 0.02 rpy=0 0 1.5708 -> xyz=1.238 -27 1.958 rpy=-3.1416 0 -1.5708
- joint joint2-1: limit lower=-3.14 upper=3.14 effort=100 velocity=1 -> lower=-3.14 upper=3.14 effort=100 velocity=10; origin xyz=3.3278 0.076034 1.9642 rpy=-1.5708 0 -1.1586 -> xyz=0 -0.6205 0.01 rpy=0 1.2343 -3.1416; parent Link2 -> Link2-0
- joint joint2-2: limit lower=-3.14 upper=3.14 effort=100 velocity=1 -> lower=-3.14 upper=3.14 effort=100 velocity=10; origin xyz=3.8796 4.0461 1.3914 rpy=-3.1416 0.35518 0.41215 -> xyz=-0.038003 0.242 0.18 rpy=3.1416 -0.72647 1.5708; parent Link2 -> Link2-1
- joint joint2-3: limit lower=-3.14 upper=3.14 effort=100 velocity=1 -> upper=3.14 effort=100 velocity=10; origin xyz=3.3278 0.076034 1.9642 rpy=-3.1416 0.14604 0.41215 -> xyz=0 -0.008 0.8 rpy=0 0.66338 0; parent Link2 -> Link2-2
- joint joint2-4: limit lower=-3.14 upper=3.14 effort=100 velocity=1 -> lower=-3.14 upper=3.14 effort=100 velocity=10; origin xyz=3.3011 0.18992 -0.55843 rpy=0.10111 0.14604 0.41215 -> xyz=0.2195 0.0433 0.225 rpy=0.64394 0 0; parent Link2 -> Link2-3
- joint joint2-5: limit lower=-3.14 upper=3.14 effort=100 velocity=1 -> lower=-3.14 upper=3.14 effort=100 velocity=10; origin xyz=2.7211 -0.15941 0.41481 rpy=0.20472 1.0573 0.5763 -> xyz=0.7905 -0.0655 0 rpy=0 0.78509 0; parent Link2 -> Link2-4
- joint joint2-6: limit lower=-3.14 upper=3.14 effort=100 velocity=1 -> lower=-3.14 upper=3.14 effort=100 velocity=10; origin xyz=3.9953 0.36827 0.48227 rpy=-1.2165 -1.0573 -2.5653 -> xyz=0.094 0.0655 0 rpy=1.768 0 -3.1416; parent Link2 -> Link2-5
