Commit message: 1

File: tiangong.urdf (robot description, URDF)
Before this commit: robot 天工机器人, 17 links, 16 joints
Joints:
- joint joint1-1: origin xyz=-0.0099737 -0.6255 0.0057037 rpy=0 1.22 3.1416 -> xyz=0 -0.6255 0 rpy=0 1.5708 3.1416
- joint joint1-2: origin xyz=-0.038003 0.242 0.18 rpy=0 0.0074575 -1.5708 -> xyz=-0.038003 0.242 0.18 rpy=0 -1.5708 -1.5708
- joint joint1-3: origin xyz=0 -0.008 0.8 rpy=0 -1.4541 0 -> xyz=0 -0.008 0.8 rpy=0 0 0
- joint joint1-4: origin xyz=0.0835 0.0433 0.225 rpy=-3.0285 0 0 -> xyz=0.0835 0.0433 0.225 rpy=0 0 0
- joint joint1-5: origin xyz=0.9265 -0.0353 0 rpy=0 1.4836 0 -> xyz=0.9265 -0.0353 0 rpy=0 0 0
- joint joint1-6: origin xyz=0.0940000046417269 0.0353002689417377 0 rpy=-0.367334218169828 0 -3.14159256129931 -> xyz=0.094 0.0353 0 rpy=-1.768 0 3.1416
- joint joint2-1: origin xyz=0 -0.6205 0.01 rpy=0 1.2343 -3.1416 -> xyz=0 -0.6205 0 rpy=0 1.5708 3.1416
- joint joint2-2: origin xyz=-0.038003 0.242 0.18 rpy=3.1416 -0.72647 1.5708 -> xyz=-0.038003 0.242 0.18 rpy=0 -1.5708 -1.5708
- joint joint2-3: origin xyz=0 -0.008 0.8 rpy=0 0.66338 0 -> xyz=0 -0.008 0.8 rpy=0 0 0
- joint joint2-4: origin xyz=0.2195 0.0433 0.225 rpy=0.64394 0 0 -> xyz=0.0835 0.0433 0.225 rpy=0 0 0
- joint joint2-5: origin xyz=0.7905 -0.0655 0 rpy=0 0.78509 0 -> xyz=0.7905 -0.0353 0 rpy=0 0 0
- joint joint2-6: origin xyz=0.094 0.0655 0 rpy=1.768 0 -3.1416 -> xyz=0.094 0.0353 0 rpy=-1.768 0 3.1416

Commit message: 1

File: tiangong.urdf (robot description, URDF)
Before this commit: robot 天工机器人, 17 links, 16 joints
Joints:
- joint joint1-6: origin xyz=0.094 0.0353 0 rpy=-1.768 0 3.1416 -> xyz=0.094 0.0353 0 rpy=0 0 3.1416
- joint joint2-6: origin xyz=0.094 0.0353 0 rpy=-1.768 0 3.1416 -> xyz=0.094 0.0353 0 rpy=0 0 3.1416

Commit message: 1

File: tiangong.urdf (robot description, URDF)
Before this commit: robot 天工机器人, 17 links, 16 joints
Joints:
- joint joint1-2: axis 0 1 0 -> 0 -1 0
- joint joint2-2: axis 0 1 0 -> 0 -1 0

Commit message: 1

File: tiangong.urdf (robot description, URDF)
Before this commit: robot 天工机器人, 17 links, 16 joints
Joints:
- joint joint1: limit lower=0 upper=14 effort=0 velocity=0 -> lower=0.1 upper=14 effort=0 velocity=0
- joint joint1-0: limit lower=0 upper=1.7 effort=0 velocity=0 -> lower=-1.38 upper=-0.1 effort=0 velocity=0; origin xyz=-0.0057039 3.1015 -2.5569 rpy=-1.5708 0 -1.5708 -> xyz=-0.0057039 1.8015 -2.5569 rpy=-1.5708 0 -1.5708
- joint joint1-1: axis 0 -1 0 -> 0 1 0
